File: FTNano.kicad_sch (KiCad schematic)
At the start: 35 parts, among them CN1 AFC10-S04QCA-00, J1 Conn_01x15_Pin, J2 Conn_01x15_Pin, Q1 2N7002DW-7-F, SW1 GT-TC029B-H020-L1N, U1 ATmega328P-MU, U2 CH340K, U3 ME6214A50M3G, U4 ME6211C33R5G, X1 CSTCE16M0V53-R0

Commit message: fix qwiic, add tvs
Parts:
- removed C10: 4.7u, Capacitor_SMD:C_0402_1005Metric, symbol Device:C
- removed D1: 1N5819WS S4, nano:SOD-323_L1.6-W1.3-LS2.7-RD, symbol nano:1N5819WSS4
- removed R6: 5.1k, Resistor_SMD:R_0402_1005Metric, symbol Device:R
- removed USB1: TYPE-C 16PIN 2MD(073), nano:USB-C-SMD_TYPE-C-6PIN-2MD-073, symbol nano:TYPE-C16PIN2MD(073)
- added D1: 1N5819WS, Diode_SMD:D_SOD-323, symbol Diode:1N5819WS
- added J3: USB_C_Receptacle_USB2.0_16P, Connector_USB:USB_C_Receptacle_G-Switch_GT-USB-7010ASV, symbol Connector:USB_C_Receptacle_USB2.0_16P
- added TV1: PRTR5V0U2X, Package_TO_SOT_SMD:SOT-143, symbol Power_Protection:PRTR5V0U2X
- C6, C7, C8: footprint Capacitor_SMD:C_0805_2012Metric -> Capacitor_SMD:C_0603_1608Metric
- R4: value 1M -> 5.1k
Connections:
- net +3.3V: now also CN1.2; no longer CN1.3
- net +5V: now also D1.1 (K)
- net DN: now also J3.A7 (D-), J3.B7 (D-), TV1.2 (I/O1)
- net DP: now also J3.A6 (D+), J3.B6 (D+), TV1.3 (I/O2)
- net GND: now also CN1.1, R5.2, J3.A1 (GND), J3.A12 (GND), J3.B1 (GND), J3.B12 (GND), J3.S1 (SHIELD); no longer CN1.4, R5.1
- net SCL: now also CN1.4; no longer CN1.1
- net SDA: now also CN1.3; no longer CN1.2
- net VBUS: now also D1.2 (A), J3.A4 (VBUS), J3.A9 (VBUS), J3.B4 (VBUS), J3.B9 (VBUS), TV1.4 (VCC)
- net at R4.1: now also J3.A5 (CC1)
- new net: J3.B5 (CC2), R5.1
Other:
- moved on the sheet: CN1

Commit message: fix led
Parts:
- removed U3: ME6214A50M3G, nano:SOT-23-3_L2.9-W1.6-P1.90-LS2.8-BR, symbol nano:ME6214A50M3G
- added U5: SPX3819M5-L-5-0, Package_TO_SOT_SMD:SOT-23-5, symbol Regulator_Linear:SPX3819M5-L-5-0
- RN1, RN2: value 2.2k -> 4.7k
Connections:
- net +5V: now also C7.2, U5.5 (OUT); no longer C7.1
- net GND: now also C6.1, C7.1, TV1.1 (GND), U5.2 (GND); no longer C6.2, C7.2
- net VDC: now also C6.2, U5.1 (IN), U5.3 (EN); no longer C6.1
- no-connect marks 7 -> 8
Other:
- moved on the sheet: C6, C7
